Commit message: wi tra_controller_balance(可懸掛用walking追點)

File: urdf/bipedal_floating.xacro (robot description, xacro)
@@ -4,9 +4,9 @@
 <xacro:include filename="$(find bipedal_floating_description)/urdf/bipedal_floating.trans" />
 <xacro:include filename="$(find bipedal_floating_description)/urdf/bipedal_floating.gazebo" />
-<link name="world"/>
+<!-- <link name="world"/>
 <joint name="fixed" type="fixed">
   <parent link="world"/>
   <child link="base_link"/>
-</joint>
+</joint> -->
 <link name="l_foot"/>
 <joint name="l_foot_joint" type="fixed">
@@ -380,5 +380,5 @@
     </command_interface>
     <command_interface name="effort"/>
-    <command_interface name="velocity"/>
+    <!-- <command_interface name="velocity"/> -->
     <state_interface name="position"/>
     <state_interface name="velocity"/>
@@ -390,5 +390,5 @@
     </command_interface>
     <command_interface name="effort"/>
-    <command_interface name="velocity"/>
+    <!-- <command_interface name="velocity"/> -->
     <state_interface name="position"/>
     <state_interface name="velocity"/>
@@ -400,5 +400,5 @@
     </command_interface>
     <command_interface name="effort"/>
-    <command_interface name="velocity"/>
+    <!-- <command_interface name="velocity"/> -->
     <state_interface name="position"/>
     <state_interface name="velocity"/>
@@ -410,5 +410,5 @@
     </command_interface>
     <command_interface name="effort"/>
-    <command_interface name="velocity"/>
+    <!-- <command_interface name="velocity"/> -->
     <state_interface name="position"/>
     <state_interface name="velocity"/>
@@ -420,5 +420,5 @@
     </command_interface>
     <command_interface name="effort"/>
-    <command_interface name="velocity"/>
+    <!-- <command_interface name="velocity"/> -->
     <state_interface name="position"/>
     <state_interface name="velocity"/>
@@ -430,5 +430,5 @@
     </command_interface>
     <command_interface name="effort"/>
-    <command_interface name="velocity"/>
+    <!-- <command_interface name="velocity"/> -->
     <state_interface name="position"/>
     <state_interface name="velocity"/>
@@ -440,5 +440,5 @@
     </command_interface>
     <command_interface name="effort"/>
-    <command_interface name="velocity"/>
+    <!-- <command_interface name="velocity"/> -->
     <state_interface name="position"/>
     <state_interface name="velocity"/>
@@ -450,5 +450,5 @@
     </command_interface>
     <command_interface name="effort"/>
-    <command_interface name="velocity"/>
+    <!-- <command_interface name="velocity"/> -->
     <state_interface name="position"/>
     <state_interface name="velocity"/>
@@ -460,5 +460,5 @@
     </command_interface>
     <command_interface name="effort"/>
-    <command_interface name="velocity"/>
+    <!-- <command_interface name="velocity"/> -->
     <state_interface name="position"/>
     <state_interface name="velocity"/>
@@ -470,5 +470,5 @@
     </command_interface>
     <command_interface name="effort"/>
-    <command_interface name="velocity"/>
+    <!-- <command_interface name="velocity"/> -->
     <state_interface name="position"/>
     <state_interface name="velocity"/>
@@ -480,5 +480,5 @@
     </command_interface>
     <command_interface name="effort"/>
-    <command_interface name="velocity"/>
+    <!-- <command_interface name="velocity"/> -->
     <state_interface name="position"/>
     <state_interface name="velocity"/>
@@ -490,5 +490,5 @@
     </command_interface>
     <command_interface name="effort"/>
-    <command_interface name="velocity"/>
+    <!-- <command_interface name="velocity"/> -->
     <state_interface name="position"/>
     <state_interface name="velocity"/>
@@ -499,5 +499,5 @@
   <plugin filename="libgazebo_ros2_control.so" name="gazebo_ros2_control">
     <robot_sim_type>gazebo_ros2_control/GazeboSystem</robot_sim_type>
-    <parameters>$(find bipedal_floating_description)/config/effort_controller.yaml</parameters>
+    <parameters>$(find bipedal_floating_description)/config/trajectory_controller.yaml</parameters>
     <!-- <parameters>$(find bipedal_floating_description)/config/velocity_controller.yaml</parameters> -->
   </plugin>

Commit message: 改effort_controller+damping (可雙腳平衡)

File: urdf/bipedal_floating.xacro (robot description, xacro)
@@ -292,4 +292,5 @@
   <child link="l_hip_yaw_1"/>
   <axis xyz="1.0 0.0 0.0"/>
+  <dynamics damping="0.2" friction="0.5"/>
   <limit upper="0.523599" lower="-0.523599" effort="100" velocity="100"/>
 </joint>
@@ -299,4 +300,5 @@
   <child link="l_hip_pitch_1"/>
   <axis xyz="0.0 0.0 1.0"/>
+  <dynamics damping="0.2" friction="0.5"/>
   <limit upper="0.523599" lower="-0.523599" effort="100" velocity="100"/>
 </joint>
@@ -306,4 +308,5 @@
   <child link="l_thigh_1"/>
   <axis xyz="0.0 1.0 -0.0"/>
+  <dynamics damping="0.2" friction="0.5"/>
   <limit upper="1.570796" lower="-1.570796" effort="100" velocity="100"/>
 </joint>
@@ -313,4 +316,5 @@
   <child link="l_shank_1"/>
   <axis xyz="0.0 1.0 0.0"/>
+  <dynamics damping="0.2" friction="0.5"/>
   <limit upper="1.919862" lower="0.0" effort="100" velocity="100"/>
 </joint>
@@ -320,4 +324,5 @@
   <child link="l_ankle_1"/>
   <axis xyz="0.0 1.0 0.0"/>
+  <dynamics damping="0.2" friction="0.5"/>
   <limit upper="0.436332" lower="-0.436332" effort="100" velocity="100"/>
 </joint>
@@ -327,4 +332,5 @@
   <child link="l_foot_1"/>
   <axis xyz="1.0 0.0 -0.0"/>
+  <dynamics damping="0.2" friction="0.5"/>
   <limit upper="0.436332" lower="-0.436332" effort="100" velocity="100"/>
 </joint>
@@ -334,4 +340,5 @@
   <child link="r_hip_yaw_1"/>
   <axis xyz="1.0 0.0 0.0"/>
+  <dynamics damping="0.2" friction="0.5"/>
   <limit upper="0.523599" lower="-0.523599" effort="100" velocity="100"/>
 </joint>
@@ -341,4 +348,5 @@
   <child link="r_hip_pitch_1"/>
   <axis xyz="0.0 0.0 1.0"/>
+  <dynamics damping="0.2" friction="0.5"/>
   <limit upper="0.523599" lower="-0.523599" effort="100" velocity="100"/>
 </joint>
@@ -348,4 +356,5 @@
   <child link="r_thigh_1"/>
   <axis xyz="0.0 1.0 0.0"/>
+  <dynamics damping="0.2" friction="0.5"/>
   <limit upper="1.570796" lower="-1.570796" effort="100" velocity="100"/>
 </joint>
@@ -355,4 +364,5 @@
   <child link="r_shank_1"/>
   <axis xyz="0.0 1.0 0.0"/>
+  <dynamics damping="0.2" friction="0.5"/>
   <limit upper="1.919862" lower="0.0" effort="100" velocity="100"/>
 </joint>
@@ -362,4 +372,5 @@
   <child link="r_ankle_1"/>
   <axis xyz="0.0 1.0 -0.0"/>
+  <dynamics damping="0.2" friction="0.5"/>
   <limit upper="0.436332" lower="-0.436332" effort="100" velocity="100"/>
 </joint>
@@ -369,4 +380,5 @@
   <child link="r_foot_1"/>
   <axis xyz="1.0 0.0 -0.0"/>
+  <dynamics damping="0.2" friction="0.5"/>
   <limit upper="0.436332" lower="-0.436332" effort="100" velocity="100"/>
 </joint>
@@ -501,4 +513,5 @@
     <parameters>$(find bipedal_floating_description)/config/trajectory_controller.yaml</parameters>
     <!-- <parameters>$(find bipedal_floating_description)/config/velocity_controller.yaml</parameters> -->
+    <parameters>$(find bipedal_floating_description)/config/effort_controller.yaml</parameters>
   </plugin>
   <plugin name="gazebo_link_attacher" filename="libgazebo_link_attacher.so"/>

Commit message: can balance by effort

File: urdf/bipedal_floating.xacro (robot description, xacro)
@@ -292,5 +292,5 @@
   <child link="l_hip_yaw_1"/>
   <axis xyz="1.0 0.0 0.0"/>
-  <dynamics damping="0.2" friction="0.5"/>
+  <dynamics damping="0.25" friction="0.5"/>
   <limit upper="0.523599" lower="-0.523599" effort="100" velocity="100"/>
 </joint>
@@ -300,5 +300,5 @@
   <child link="l_hip_pitch_1"/>
   <axis xyz="0.0 0.0 1.0"/>
-  <dynamics damping="0.2" friction="0.5"/>
+  <dynamics damping="0.25" friction="0.5"/>
   <limit upper="0.523599" lower="-0.523599" effort="100" velocity="100"/>
 </joint>
@@ -308,5 +308,5 @@
   <child link="l_thigh_1"/>
   <axis xyz="0.0 1.0 -0.0"/>
-  <dynamics damping="0.2" friction="0.5"/>
+  <dynamics damping="0.25" friction="0.5"/>
   <limit upper="1.570796" lower="-1.570796" effort="100" velocity="100"/>
 </joint>
@@ -316,5 +316,5 @@
   <child link="l_shank_1"/>
   <axis xyz="0.0 1.0 0.0"/>
-  <dynamics damping="0.2" friction="0.5"/>
+  <dynamics damping="0.25" friction="0.5"/>
   <limit upper="1.919862" lower="0.0" effort="100" velocity="100"/>
 </joint>
@@ -340,5 +340,5 @@
   <child link="r_hip_yaw_1"/>
   <axis xyz="1.0 0.0 0.0"/>
-  <dynamics damping="0.2" friction="0.5"/>
+  <dynamics damping="0.25" friction="0.5"/>
   <limit upper="0.523599" lower="-0.523599" effort="100" velocity="100"/>
 </joint>
@@ -348,5 +348,5 @@
   <child link="r_hip_pitch_1"/>
   <axis xyz="0.0 0.0 1.0"/>
-  <dynamics damping="0.2" friction="0.5"/>
+  <dynamics damping="0.25" friction="0.5"/>
   <limit upper="0.523599" lower="-0.523599" effort="100" velocity="100"/>
 </joint>
@@ -356,5 +356,5 @@
   <child link="r_thigh_1"/>
   <axis xyz="0.0 1.0 0.0"/>
-  <dynamics damping="0.2" friction="0.5"/>
+  <dynamics damping="0.25" friction="0.5"/>
   <limit upper="1.570796" lower="-1.570796" effort="100" velocity="100"/>
 </joint>
@@ -364,5 +364,5 @@
   <child link="r_shank_1"/>
   <axis xyz="0.0 1.0 0.0"/>
-  <dynamics damping="0.2" friction="0.5"/>
+  <dynamics damping="0.25" friction="0.5"/>
   <limit upper="1.919862" lower="0.0" effort="100" velocity="100"/>
 </joint>

Commit message: can walk

File: urdf/bipedal_floating.xacro (robot description, xacro)
@@ -372,5 +372,5 @@
   <child link="r_ankle_1"/>
   <axis xyz="0.0 1.0 -0.0"/>
-  <dynamics damping="0.2" friction="0.5"/>
+  <dynamics damping="0.2" friction="0.3"/>
   <limit upper="0.436332" lower="-0.436332" effort="100" velocity="100"/>
 </joint>

Commit message: norman (fixed)

File: urdf/bipedal_floating.xacro (robot description, xacro)
@@ -372,5 +372,5 @@
   <child link="r_ankle_1"/>
   <axis xyz="0.0 1.0 -0.0"/>
-  <dynamics damping="0.2" friction="0.3"/>
+  <dynamics damping="0.2" friction="0.5"/>
   <limit upper="0.436332" lower="-0.436332" effort="100" velocity="100"/>
 </joint>

Commit message: gravity_compensate

File: urdf/bipedal_floating.xacro (robot description, xacro)
@@ -332,5 +332,5 @@
   <child link="l_foot_1"/>
   <axis xyz="1.0 0.0 -0.0"/>
-  <dynamics damping="0.2" friction="0.5"/>
+  <dynamics damping="0.2" friction="1.5"/>
   <limit upper="0.436332" lower="-0.436332" effort="100" velocity="100"/>
 </joint>

Commit message: 可以走個幾步

File: urdf/bipedal_floating.xacro (robot description, xacro)
@@ -316,5 +316,5 @@
   <child link="l_shank_1"/>
   <axis xyz="0.0 1.0 0.0"/>
-  <dynamics damping="0.25" friction="0.5"/>
+  <dynamics damping="0.25" friction="0.4"/>
   <limit upper="1.919862" lower="0.0" effort="100" velocity="100"/>
 </joint>
@@ -364,5 +364,5 @@
   <child link="r_shank_1"/>
   <axis xyz="0.0 1.0 0.0"/>
-  <dynamics damping="0.25" friction="0.5"/>
+  <dynamics damping="0.25" friction="0.4"/>
   <limit upper="1.919862" lower="0.0" effort="100" velocity="100"/>
 </joint>

Commit message: 以此為主

File: urdf/bipedal_floating.xacro (robot description, xacro)
@@ -332,5 +332,5 @@
   <child link="l_foot_1"/>
   <axis xyz="1.0 0.0 -0.0"/>
-  <dynamics damping="0.2" friction="1.5"/>
+  <dynamics damping="0.2" friction="0.5"/>
   <limit upper="0.436332" lower="-0.436332" effort="100" velocity="100"/>
 </joint>

Commit message: 完成ALIP_x軌跡索取

File: urdf/bipedal_floating.xacro (robot description, xacro)
@@ -324,5 +324,5 @@
   <child link="l_ankle_1"/>
   <axis xyz="0.0 1.0 0.0"/>
-  <dynamics damping="0.2" friction="0.5"/>
+  <dynamics damping="0.0" friction="0.0"/>
   <limit upper="0.436332" lower="-0.436332" effort="100" velocity="100"/>
 </joint>

Commit message: 平衡＆給impulse

File: urdf/bipedal_floating.xacro (robot description, xacro)
@@ -308,5 +308,5 @@
   <child link="l_thigh_1"/>
   <axis xyz="0.0 1.0 -0.0"/>
-  <dynamics damping="0.25" friction="0.5"/>
+  <dynamics damping="0.25" friction="0.3"/>
   <limit upper="1.570796" lower="-1.570796" effort="100" velocity="100"/>
 </joint>

Commit message: Exp

File: urdf/bipedal_floating.xacro (robot description, xacro)
@@ -292,5 +292,5 @@
   <child link="l_hip_yaw_1"/>
   <axis xyz="1.0 0.0 0.0"/>
-  <dynamics damping="0.25" friction="0.5"/>
+  <dynamics damping="0.25" friction="0.2"/>
   <limit upper="0.523599" lower="-0.523599" effort="100" velocity="100"/>
 </joint>
@@ -308,5 +308,5 @@
   <child link="l_thigh_1"/>
   <axis xyz="0.0 1.0 -0.0"/>
-  <dynamics damping="0.25" friction="0.3"/>
+  <dynamics damping="0.25" friction="0.4"/>
   <limit upper="1.570796" lower="-1.570796" effort="100" velocity="100"/>
 </joint>
@@ -324,5 +324,5 @@
   <child link="l_ankle_1"/>
   <axis xyz="0.0 1.0 0.0"/>
-  <dynamics damping="0.0" friction="0.0"/>
+  <dynamics damping="0.0" friction="0.2"/>
   <limit upper="0.436332" lower="-0.436332" effort="100" velocity="100"/>
 </joint>
@@ -332,5 +332,5 @@
   <child link="l_foot_1"/>
   <axis xyz="1.0 0.0 -0.0"/>
-  <dynamics damping="0.2" friction="0.5"/>
+  <dynamics damping="0.2" friction="0.2"/>
   <limit upper="0.436332" lower="-0.436332" effort="100" velocity="100"/>
 </joint>
@@ -340,5 +340,5 @@
   <child link="r_hip_yaw_1"/>
   <axis xyz="1.0 0.0 0.0"/>
-  <dynamics damping="0.25" friction="0.5"/>
+  <dynamics damping="0.25" friction="0.2"/>
   <limit upper="0.523599" lower="-0.523599" effort="100" velocity="100"/>
 </joint>
@@ -372,5 +372,5 @@
   <child link="r_ankle_1"/>
   <axis xyz="0.0 1.0 -0.0"/>
-  <dynamics damping="0.2" friction="0.5"/>
+  <dynamics damping="0.2" friction="0.2"/>
   <limit upper="0.436332" lower="-0.436332" effort="100" velocity="100"/>
 </joint>
@@ -380,5 +380,5 @@
   <child link="r_foot_1"/>
   <axis xyz="1.0 0.0 -0.0"/>
-  <dynamics damping="0.2" friction="0.5"/>
+  <dynamics damping="0.2" friction="0.2"/>
   <limit upper="0.436332" lower="-0.436332" effort="100" velocity="100"/>
 </joint>

File: urdf/stance_l.xacro (robot description, xacro)
@@ -150,5 +150,5 @@
   <child link="B_UNCA10_ros_v3_1"/>
   <axis xyz="1.0 0.0 0.0"/>
-  <dynamics damping="0.0" friction="0.1"/>
+  <dynamics damping="0.0" friction="0.0"/>
   <limit upper="0.436332" lower="-0.436332" effort="100" velocity="100"/>
 </joint>
@@ -158,5 +158,5 @@
   <child link="shank_ros_v4_1"/>
   <axis xyz="0.0 1.0 0.0"/>
-  <dynamics damping="0.0" friction="0.1"/>
+  <dynamics damping="0.0" friction="0.0"/>
   <limit upper="0.436332" lower="-0.436332" effort="100" velocity="100"/>
 </joint>
@@ -166,5 +166,5 @@
   <child link="thigh_l_ros_v4_1"/>
   <axis xyz="0.0 1.0 0.0"/>
-  <dynamics damping="0.0" friction="0.05"/>
+  <dynamics damping="0.0" friction="0.0"/>
   <limit upper="0.0" lower="-1.919862" effort="100" velocity="100"/>
 </joint>
@@ -174,5 +174,5 @@
   <child link="l_hip_pitch_ros_v4_1"/>
   <axis xyz="0.0 1.0 0.0"/>
-  <dynamics damping="0.0" friction="0.05"/>
+  <dynamics damping="0.0" friction="0.0"/>
   <limit upper="1.570796" lower="-1.570796" effort="100" velocity="100"/>
 </joint>
@@ -182,5 +182,5 @@
   <child link="hip_yaw_ros_v3_1"/>
   <axis xyz="0.0 0.0 1.0"/>
-  <dynamics damping="0.0" friction="0.05"/>
+  <dynamics damping="0.0" friction="0.0"/>
   <limit upper="0.523599" lower="-0.523599" effort="100" velocity="100"/>
 </joint>
@@ -190,5 +190,5 @@
   <child link="waist_ros_v2_1"/>
   <axis xyz="1.0 0.0 0.0"/>
-  <dynamics damping="0.0" friction="0.05"/>
+  <dynamics damping="0.0" friction="0.0"/>
   <limit upper="0.523599" lower="-1.570796" effort="100" velocity="100"/>
 </joint>

Commit message: lift lef leg +change state(wi bug)

File: urdf/bipedal_floating.xacro (robot description, xacro)
@@ -308,5 +308,5 @@
   <child link="l_thigh_1"/>
   <axis xyz="0.0 1.0 -0.0"/>
-  <dynamics damping="0.25" friction="0.4"/>
+  <dynamics damping="0.25" friction="0.2"/>
   <limit upper="1.570796" lower="-1.570796" effort="100" velocity="100"/>
 </joint>
@@ -316,5 +316,5 @@
   <child link="l_shank_1"/>
   <axis xyz="0.0 1.0 0.0"/>
-  <dynamics damping="0.25" friction="0.4"/>
+  <dynamics damping="0.25" friction="0.2"/>
   <limit upper="1.919862" lower="0.0" effort="100" velocity="100"/>
 </joint>

Commit message: lift l_leg + balance+ back to center

File: urdf/bipedal_floating.xacro (robot description, xacro)
@@ -324,5 +324,5 @@
   <child link="l_ankle_1"/>
   <axis xyz="0.0 1.0 0.0"/>
-  <dynamics damping="0.0" friction="0.2"/>
+  <dynamics damping="0.2" friction="0.5"/>
   <limit upper="0.436332" lower="-0.436332" effort="100" velocity="100"/>
 </joint>
@@ -332,5 +332,5 @@
   <child link="l_foot_1"/>
   <axis xyz="1.0 0.0 -0.0"/>
-  <dynamics damping="0.2" friction="0.2"/>
+  <dynamics damping="0.2" friction="0.5"/>
   <limit upper="0.436332" lower="-0.436332" effort="100" velocity="100"/>
 </joint>

Commit message: can walk

File: urdf/bipedal_floating.xacro (robot description, xacro)
@@ -316,5 +316,5 @@
   <child link="l_shank_1"/>
   <axis xyz="0.0 1.0 0.0"/>
-  <dynamics damping="0.25" friction="0.2"/>
+  <dynamics damping="0.25" friction="0.4"/>
   <limit upper="1.919862" lower="0.0" effort="100" velocity="100"/>
 </joint>
@@ -372,5 +372,5 @@
   <child link="r_ankle_1"/>
   <axis xyz="0.0 1.0 -0.0"/>
-  <dynamics damping="0.2" friction="0.2"/>
+  <dynamics damping="0.2" friction="0.5"/>
   <limit upper="0.436332" lower="-0.436332" effort="100" velocity="100"/>
 </joint>
@@ -380,5 +380,5 @@
   <child link="r_foot_1"/>
   <axis xyz="1.0 0.0 -0.0"/>
-  <dynamics damping="0.2" friction="0.2"/>
+  <dynamics damping="0.2" friction="0.5"/>
   <limit upper="0.436332" lower="-0.436332" effort="100" velocity="100"/>
 </joint>

Commit message: need to add position filter and v_limit (RTF=0.8)

File: urdf/bipedal_floating.xacro (robot description, xacro)
@@ -293,5 +293,5 @@
   <axis xyz="1.0 0.0 0.0"/>
   <dynamics damping="0.25" friction="0.2"/>
-  <limit upper="0.523599" lower="-0.523599" effort="100" velocity="100"/>
+  <limit upper="0.523599" lower="-0.523599" effort="15" velocity="45"/>
 </joint>
 <joint name="L_Hip_Yaw" type="revolute">
@@ -301,5 +301,5 @@
   <axis xyz="0.0 0.0 1.0"/>
   <dynamics damping="0.25" friction="0.5"/>
-  <limit upper="0.523599" lower="-0.523599" effort="100" velocity="100"/>
+  <limit upper="0.523599" lower="-0.523599" effort="15" velocity="45"/>
 </joint>
 <joint name="L_Hip_Pitch" type="revolute">
@@ -309,5 +309,5 @@
   <axis xyz="0.0 1.0 -0.0"/>
   <dynamics damping="0.25" friction="0.2"/>
-  <limit upper="1.570796" lower="-1.570796" effort="100" velocity="100"/>
+  <limit upper="1.570796" lower="-1.570796" effort="15" velocity="45"/>
 </joint>
 <joint name="L_Knee_Pitch" type="revolute">
@@ -317,5 +317,5 @@
   <axis xyz="0.0 1.0 0.0"/>
   <dynamics damping="0.25" friction="0.4"/>
-  <limit upper="1.919862" lower="0.0" effort="100" velocity="100"/>
+  <limit upper="1.919862" lower="0.0" effort="15" velocity="45"/>
 </joint>
 <joint name="L_Ankle_Pitch" type="revolute">
@@ -325,5 +325,5 @@
   <axis xyz="0.0 1.0 0.0"/>
   <dynamics damping="0.2" friction="0.5"/>
-  <limit upper="0.436332" lower="-0.436332" effort="100" velocity="100"/>
+  <limit upper="0.436332" lower="-0.436332" effort="15" velocity="45"/>
 </joint>
 <joint name="L_Ankle_Roll" type="revolute">
@@ -333,5 +333,5 @@
   <axis xyz="1.0 0.0 -0.0"/>
   <dynamics damping="0.2" friction="0.5"/>
-  <limit upper="0.436332" lower="-0.436332" effort="100" velocity="100"/>
+  <limit upper="0.436332" lower="-0.436332" effort="15" velocity="45"/>
 </joint>
 <joint name="R_Hip_Roll" type="revolute">
@@ -341,5 +341,5 @@
   <axis xyz="1.0 0.0 0.0"/>
   <dynamics damping="0.25" friction="0.2"/>
-  <limit upper="0.523599" lower="-0.523599" effort="100" velocity="100"/>
+  <limit upper="0.523599" lower="-0.523599" effort="15" velocity="45"/>
 </joint>
 <joint name="R_Hip_Yaw" type="revolute">
@@ -349,5 +349,5 @@
   <axis xyz="0.0 0.0 1.0"/>
   <dynamics damping="0.25" friction="0.5"/>
-  <limit upper="0.523599" lower="-0.523599" effort="100" velocity="100"/>
+  <limit upper="0.523599" lower="-0.523599" effort="15" velocity="45"/>
 </joint>
 <joint name="R_Hip_Pitch" type="revolute">
@@ -357,5 +357,5 @@
   <axis xyz="0.0 1.0 0.0"/>
   <dynamics damping="0.25" friction="0.5"/>
-  <limit upper="1.570796" lower="-1.570796" effort="100" velocity="100"/>
+  <limit upper="1.570796" lower="-1.570796" effort="15" velocity="45"/>
 </joint>
 <joint name="R_Knee_Pitch" type="revolute">
@@ -365,5 +365,5 @@
   <axis xyz="0.0 1.0 0.0"/>
   <dynamics damping="0.25" friction="0.4"/>
-  <limit upper="1.919862" lower="0.0" effort="100" velocity="100"/>
+  <limit upper="1.919862" lower="0.0" effort="15" velocity="45"/>
 </joint>
 <joint name="R_Ankle_Pitch" type="revolute">
@@ -373,5 +373,5 @@
   <axis xyz="0.0 1.0 -0.0"/>
   <dynamics damping="0.2" friction="0.5"/>
-  <limit upper="0.436332" lower="-0.436332" effort="100" velocity="100"/>
+  <limit upper="0.436332" lower="-0.436332" effort="15" velocity="45"/>
 </joint>
 <joint name="R_Ankle_Roll" type="revolute">
@@ -381,5 +381,5 @@
   <axis xyz="1.0 0.0 -0.0"/>
   <dynamics damping="0.2" friction="0.5"/>
-  <limit upper="0.436332" lower="-0.436332" effort="100" velocity="100"/>
+  <limit upper="0.436332" lower="-0.436332" effort="15" velocity="45"/>
 </joint>
 <ros2_control name="GazeboSystem" type="system">

Commit message: 往後走？？？

File: urdf/bipedal_floating.xacro (robot description, xacro)
@@ -292,5 +292,5 @@
   <child link="l_hip_yaw_1"/>
   <axis xyz="1.0 0.0 0.0"/>
-  <dynamics damping="0.25" friction="0.2"/>
+  <dynamics damping="0.5" friction="0.2"/>
   <limit upper="0.523599" lower="-0.523599" effort="15" velocity="45"/>
 </joint>
@@ -300,5 +300,5 @@
   <child link="l_hip_pitch_1"/>
   <axis xyz="0.0 0.0 1.0"/>
-  <dynamics damping="0.25" friction="0.5"/>
+  <dynamics damping="0.5" friction="0.2"/>
   <limit upper="0.523599" lower="-0.523599" effort="15" velocity="45"/>
 </joint>
@@ -308,5 +308,5 @@
   <child link="l_thigh_1"/>
   <axis xyz="0.0 1.0 -0.0"/>
-  <dynamics damping="0.25" friction="0.2"/>
+  <dynamics damping="0.5" friction="0.2"/>
   <limit upper="1.570796" lower="-1.570796" effort="15" velocity="45"/>
 </joint>
@@ -316,5 +316,5 @@
   <child link="l_shank_1"/>
   <axis xyz="0.0 1.0 0.0"/>
-  <dynamics damping="0.25" friction="0.4"/>
+  <dynamics damping="0.25" friction="0.2"/>
   <limit upper="1.919862" lower="0.0" effort="15" velocity="45"/>
 </joint>
@@ -340,5 +340,5 @@
   <child link="r_hip_yaw_1"/>
   <axis xyz="1.0 0.0 0.0"/>
-  <dynamics damping="0.25" friction="0.2"/>
+  <dynamics damping="0.5" friction="0.2"/>
   <limit upper="0.523599" lower="-0.523599" effort="15" velocity="45"/>
 </joint>
@@ -348,5 +348,5 @@
   <child link="r_hip_pitch_1"/>
   <axis xyz="0.0 0.0 1.0"/>
-  <dynamics damping="0.25" friction="0.5"/>
+  <dynamics damping="0.5" friction="0.2"/>
   <limit upper="0.523599" lower="-0.523599" effort="15" velocity="45"/>
 </joint>
@@ -356,5 +356,5 @@
   <child link="r_thigh_1"/>
   <axis xyz="0.0 1.0 0.0"/>
-  <dynamics damping="0.25" friction="0.5"/>
+  <dynamics damping="0.5" friction="0.2"/>
   <limit upper="1.570796" lower="-1.570796" effort="15" velocity="45"/>
 </joint>
@@ -364,5 +364,5 @@
   <child link="r_shank_1"/>
   <axis xyz="0.0 1.0 0.0"/>
-  <dynamics damping="0.25" friction="0.4"/>
+  <dynamics damping="0.25" friction="0.2"/>
   <limit upper="1.919862" lower="0.0" effort="15" velocity="45"/>
 </joint>
