Commit message: 需要處理碰撞瞬間

File: urdf/bipedal_floating.xacro (robot description, xacro)
@@ -292,5 +292,5 @@
   <child link="l_hip_yaw_1"/>
   <axis xyz="1.0 0.0 0.0"/>
-  <dynamics damping="0.5" friction="0.2"/>
+  <dynamics damping="1" friction="0.2"/>
   <limit upper="0.523599" lower="-0.523599" effort="15" velocity="45"/>
 </joint>
@@ -300,5 +300,5 @@
   <child link="l_hip_pitch_1"/>
   <axis xyz="0.0 0.0 1.0"/>
-  <dynamics damping="0.5" friction="0.2"/>
+  <dynamics damping="1" friction="0.2"/>
   <limit upper="0.523599" lower="-0.523599" effort="15" velocity="45"/>
 </joint>
@@ -308,5 +308,5 @@
   <child link="l_thigh_1"/>
   <axis xyz="0.0 1.0 -0.0"/>
-  <dynamics damping="0.5" friction="0.2"/>
+  <dynamics damping="1" friction="0.2"/>
   <limit upper="1.570796" lower="-1.570796" effort="15" velocity="45"/>
 </joint>
@@ -324,5 +324,5 @@
   <child link="l_ankle_1"/>
   <axis xyz="0.0 1.0 0.0"/>
-  <dynamics damping="0.2" friction="0.5"/>
+  <dynamics damping="0.2" friction="0.2"/>
   <limit upper="0.436332" lower="-0.436332" effort="15" velocity="45"/>
 </joint>
@@ -332,5 +332,5 @@
   <child link="l_foot_1"/>
   <axis xyz="1.0 0.0 -0.0"/>
-  <dynamics damping="0.2" friction="0.5"/>
+  <dynamics damping="0.2" friction="0.2"/>
   <limit upper="0.436332" lower="-0.436332" effort="15" velocity="45"/>
 </joint>
@@ -340,5 +340,5 @@
   <child link="r_hip_yaw_1"/>
   <axis xyz="1.0 0.0 0.0"/>
-  <dynamics damping="0.5" friction="0.2"/>
+  <dynamics damping="1" friction="0.2"/>
   <limit upper="0.523599" lower="-0.523599" effort="15" velocity="45"/>
 </joint>
@@ -348,5 +348,5 @@
   <child link="r_hip_pitch_1"/>
   <axis xyz="0.0 0.0 1.0"/>
-  <dynamics damping="0.5" friction="0.2"/>
+  <dynamics damping="1" friction="0.2"/>
   <limit upper="0.523599" lower="-0.523599" effort="15" velocity="45"/>
 </joint>
@@ -356,5 +356,5 @@
   <child link="r_thigh_1"/>
   <axis xyz="0.0 1.0 0.0"/>
-  <dynamics damping="0.5" friction="0.2"/>
+  <dynamics damping="1" friction="0.2"/>
   <limit upper="1.570796" lower="-1.570796" effort="15" velocity="45"/>
 </joint>
@@ -372,5 +372,5 @@
   <child link="r_ankle_1"/>
   <axis xyz="0.0 1.0 -0.0"/>
-  <dynamics damping="0.2" friction="0.5"/>
+  <dynamics damping="0.2" friction="0.2"/>
   <limit upper="0.436332" lower="-0.436332" effort="15" velocity="45"/>
 </joint>
@@ -380,5 +380,5 @@
   <child link="r_foot_1"/>
   <axis xyz="1.0 0.0 -0.0"/>
-  <dynamics damping="0.2" friction="0.5"/>
+  <dynamics damping="0.2" friction="0.2"/>
   <limit upper="0.436332" lower="-0.436332" effort="15" velocity="45"/>
 </joint>

Commit message: add wf

File: urdf/bipedal_floating.xacro (robot description, xacro)
@@ -4,9 +4,4 @@
 <xacro:include filename="$(find bipedal_floating_description)/urdf/bipedal_floating.trans" />
 <xacro:include filename="$(find bipedal_floating_description)/urdf/bipedal_floating.gazebo" />
-<!-- <link name="world"/>
-<joint name="fixed" type="fixed">
-  <parent link="world"/>
-  <child link="base_link"/>
-</joint> -->
 <link name="l_foot"/>
 <joint name="l_foot_joint" type="fixed">
@@ -516,4 +511,12 @@
   </plugin>
   <plugin name="gazebo_link_attacher" filename="libgazebo_link_attacher.so"/>
+  <plugin name="p3d_base_controller" filename="libgazebo_ros_p3d.so">
+    <update_rate>500.0</update_rate>
+    <body_name>base_link</body_name>
+    <frame_name>world</frame_name>
+    <gaussian_noise>0.0</gaussian_noise>
+    <xyz_offset>0 0 0</xyz_offset>
+    <rpy_offset>0 0 0</rpy_offset>
+  </plugin>
 </gazebo>
 </robot>

Commit message: not good

File: urdf/bipedal_floating.xacro (robot description, xacro)
@@ -319,5 +319,5 @@
   <child link="l_ankle_1"/>
   <axis xyz="0.0 1.0 0.0"/>
-  <dynamics damping="0.2" friction="0.2"/>
+  <dynamics damping="0.1" friction="0.2"/>
   <limit upper="0.436332" lower="-0.436332" effort="15" velocity="45"/>
 </joint>
@@ -327,5 +327,5 @@
   <child link="l_foot_1"/>
   <axis xyz="1.0 0.0 -0.0"/>
-  <dynamics damping="0.2" friction="0.2"/>
+  <dynamics damping="0.1" friction="0.2"/>
   <limit upper="0.436332" lower="-0.436332" effort="15" velocity="45"/>
 </joint>
@@ -367,5 +367,5 @@
   <child link="r_ankle_1"/>
   <axis xyz="0.0 1.0 -0.0"/>
-  <dynamics damping="0.2" friction="0.2"/>
+  <dynamics damping="0.1" friction="0.2"/>
   <limit upper="0.436332" lower="-0.436332" effort="15" velocity="45"/>
 </joint>
@@ -375,5 +375,5 @@
   <child link="r_foot_1"/>
   <axis xyz="1.0 0.0 -0.0"/>
-  <dynamics damping="0.2" friction="0.2"/>
+  <dynamics damping="0.1" friction="0.2"/>
   <limit upper="0.436332" lower="-0.436332" effort="15" velocity="45"/>
 </joint>

Commit message: 改0.15一樣會翻

File: urdf/bipedal_floating.xacro (robot description, xacro)
@@ -319,5 +319,5 @@
   <child link="l_ankle_1"/>
   <axis xyz="0.0 1.0 0.0"/>
-  <dynamics damping="0.1" friction="0.2"/>
+  <dynamics damping="0.05" friction="0.2"/>
   <limit upper="0.436332" lower="-0.436332" effort="15" velocity="45"/>
 </joint>
@@ -327,5 +327,5 @@
   <child link="l_foot_1"/>
   <axis xyz="1.0 0.0 -0.0"/>
-  <dynamics damping="0.1" friction="0.2"/>
+  <dynamics damping="0.05" friction="0.2"/>
   <limit upper="0.436332" lower="-0.436332" effort="15" velocity="45"/>
 </joint>
@@ -367,5 +367,5 @@
   <child link="r_ankle_1"/>
   <axis xyz="0.0 1.0 -0.0"/>
-  <dynamics damping="0.1" friction="0.2"/>
+  <dynamics damping="0.05" friction="0.2"/>
   <limit upper="0.436332" lower="-0.436332" effort="15" velocity="45"/>
 </joint>
@@ -375,5 +375,5 @@
   <child link="r_foot_1"/>
   <axis xyz="1.0 0.0 -0.0"/>
-  <dynamics damping="0.1" friction="0.2"/>
+  <dynamics damping="0.05" friction="0.2"/>
   <limit upper="0.436332" lower="-0.436332" effort="15" velocity="45"/>
 </joint>
