Commit message: gazebo&pink

File: urdf/bipedal_floating.pin.urdf (robot description, URDF)
Before this commit: robot bipedal_floating, 13 links, 12 joints
Links:
- link base_link: geometry collision mesh filename=file:///home/ldsc/ros2_ws/src/bipedal_floating_description/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 scale=0.001 0.001 0.001; visual mesh filename=file:///home/ldsc/ros2_ws/src/bipedal_floating_description/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 scale=0.001 0.001 0.001
- link l_ankle_1: geometry collision mesh filename=file:///home/ldsc/ros2_ws/src/bipedal_floating_description/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 scale=0.001 0.001 0.001; visual mesh filename=file:///home/ldsc/ros2_ws/src/bipedal_floating_description/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 scale=0.001 0.001 0.001
- link l_foot_1: geometry collision mesh filename=file:///home/ldsc/ros2_ws/src/bipedal_floating_description/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 scale=0.001 0.001 0.001; visual mesh filename=file:///home/ldsc/ros2_ws/src/bipedal_floating_description/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 scale=0.001 0.001 0.001
- link l_hip_pitch_1: geometry collision mesh filename=file:///home/ldsc/ros2_ws/src/bipedal_floating_description/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 scale=0.001 0.001 0.001; visual mesh filename=file:///home/ldsc/ros2_ws/src/bipedal_floating_description/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 scale=0.001 0.001 0.001
- link l_hip_yaw_1: geometry collision mesh filename=file:///home/ldsc/ros2_ws/src/bipedal_floating_description/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 scale=0.001 0.001 0.001; visual mesh filename=file:///home/ldsc/ros2_ws/src/bipedal_floating_description/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 scale=0.001 0.001 0.001
- link l_shank_1: geometry collision mesh filename=file:///home/ldsc/ros2_ws/src/bipedal_floating_description/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 scale=0.001 0.001 0.001; visual mesh filename=file:///home/ldsc/ros2_ws/src/bipedal_floating_description/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 scale=0.001 0.001 0.001
- link l_thigh_1: geometry collision mesh filename=file:///home/ldsc/ros2_ws/src/bipedal_floating_description/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 scale=0.001 0.001 0.001; visual mesh filename=file:///home/ldsc/ros2_ws/src/bipedal_floating_description/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 scale=0.001 0.001 0.001
- link r_ankle_1: geometry collision mesh filename=file:///home/ldsc/ros2_ws/src/bipedal_floating_description/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 scale=0.001 0.001 0.001; visual mesh filename=file:///home/ldsc/ros2_ws/src/bipedal_floating_description/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 scale=0.001 0.001 0.001
- link r_foot_1: geometry collision mesh filename=file:///home/ldsc/ros2_ws/src/bipedal_floating_description/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 scale=0.001 0.001 0.001; visual mesh filename=file:///home/ldsc/ros2_ws/src/bipedal_floating_description/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 scale=0.001 0.001 0.001
- link r_hip_pitch_1: geometry collision mesh filename=file:///home/ldsc/ros2_ws/src/bipedal_floating_description/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 scale=0.001 0.001 0.001; visual mesh filename=file:///home/ldsc/ros2_ws/src/bipedal_floating_description/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 scale=0.001 0.001 0.001
- link r_hip_yaw_1: geometry collision mesh filename=file:///home/ldsc/ros2_ws/src/bipedal_floating_description/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 scale=0.001 0.001 0.001; visual mesh filename=file:///home/ldsc/ros2_ws/src/bipedal_floating_description/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 scale=0.001 0.001 0.001
- link r_shank_1: geometry collision mesh filename=file:///home/ldsc/ros2_ws/src/bipedal_floating_description/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 scale=0.001 0.001 0.001; visual mesh filename=file:///home/ldsc/ros2_ws/src/bipedal_floating_description/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 scale=0.001 0.001 0.001
- link r_thigh_1: geometry collision mesh filename=file:///home/ldsc/ros2_ws/src/bipedal_floating_description/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 scale=0.001 0.001 0.001; visual mesh filename=file:///home/ldsc/ros2_ws/src/bipedal_floating_description/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 scale=0.001 0.001 0.001

Commit message: 無結果

File: urdf/bipedal_floating.pin.urdf (robot description, URDF)
Before this commit: robot bipedal_floating, 13 links, 12 joints
Links:
- added link pelvis_link, mass 0; collision box size=0 0 0; visual box size=0 0 0
Joints:
- added joint dummy_joint: type fixed, parent l_hip_yaw_1, child pelvis_link, origin xyz=0 -0.049 0 rpy=0 0 0

File: urdf/bipedal_floating.xacro (robot description, xacro)
@@ -4,4 +4,25 @@
 <xacro:include filename="$(find bipedal_floating_description)/urdf/bipedal_floating.trans" />
 <xacro:include filename="$(find bipedal_floating_description)/urdf/bipedal_floating.gazebo" />
+<link name="pelvis_link">
+  <visual>
+    <geometry>
+      <box size="0 0 0"/>
+    </geometry>
+  </visual>
+  <collision>
+    <geometry>
+      <box size="0 0 0"/>
+    </geometry>
+  </collision>
+  <inertial>
+    <mass value="0"/>
+    <inertia ixx="0" ixy="0" ixz="0" iyy="0" iyz="0" izz="0"/>
+  </inertial>
+</link>
+<joint name="dummy_joint" type="fixed">
+  <parent link="l_hip_yaw_1"/>
+  <child link="pelvis_link"/>
+  <origin xyz="0 -0.049 0" rpy="0 0 0"/>
+</joint>
 <link name="base_link">
   <inertial>

Commit message: can get relative axis

File: urdf/bipedal_floating.pin.urdf (robot description, URDF)
Before this commit: robot bipedal_floating, 14 links, 13 joints
Joints:
- joint dummy_joint: origin xyz=0 -0.049 0 rpy=0 0 0 -> xyz=0 0 0.598 rpy=0 0 0; parent l_hip_yaw_1 -> base_link

File: urdf/bipedal_floating.xacro (robot description, xacro)
@@ -4,4 +4,9 @@
 <xacro:include filename="$(find bipedal_floating_description)/urdf/bipedal_floating.trans" />
 <xacro:include filename="$(find bipedal_floating_description)/urdf/bipedal_floating.gazebo" />
+<link name="world"/>
+<joint name="fixed" type="fixed">
+  <parent link="world"/>
+  <child link="base_link"/>
+</joint>
 <link name="pelvis_link">
   <visual>

Commit message: jaco

File: urdf/bipedal_floating.pin.urdf (robot description, URDF)
Before this commit: robot bipedal_floating, 14 links, 13 joints
Links:
- added link l_foot
- added link r_foot
- link pelvis_link: mass 0 -> None; geometry 
Joints:
- removed joint dummy_joint
- added joint l_foot_joint: type fixed, parent l_foot_1, child l_foot, origin xyz=0 0 -0.026 rpy=0 0 0
- added joint pelvis_joint: type fixed, parent base_link, child pelvis_link, origin xyz=0 0 0.598 rpy=0 0 0
- added joint r_foot_joint: type fixed, parent r_foot_1, child r_foot, origin xyz=0 0 -0.026 rpy=0 0 0

File: urdf/bipedal_floating.xacro (robot description, xacro)
@@ -9,24 +9,21 @@
   <child link="base_link"/>
 </joint>
-<link name="pelvis_link">
-  <visual>
-    <geometry>
-      <box size="0 0 0"/>
-    </geometry>
-  </visual>
-  <collision>
-    <geometry>
-      <box size="0 0 0"/>
-    </geometry>
-  </collision>
-  <inertial>
-    <mass value="0"/>
-    <inertia ixx="0" ixy="0" ixz="0" iyy="0" iyz="0" izz="0"/>
-  </inertial>
-</link>
-<joint name="dummy_joint" type="fixed">
-  <parent link="l_hip_yaw_1"/>
+<link name="l_foot"/>
+<joint name="l_foot_joint" type="fixed">
+  <parent link="l_foot_1"/>
+  <child link="l_foot"/>
+  <origin xyz="0 0 -0.026" rpy="0 0 0"/>
+</joint>
+<link name="r_foot"/>
+<joint name="r_foot_joint" type="fixed">
+  <parent link="r_foot_1"/>
+  <child link="r_foot"/>
+  <origin xyz="0 0 -0.026" rpy="0 0 0"/>
+</joint>
+<link name="pelvis_link"/>
+<joint name="pelvis_joint" type="fixed">
+  <parent link="base_link"/>
   <child link="pelvis_link"/>
-  <origin xyz="0 -0.049 0" rpy="0 0 0"/>
+  <origin xyz="0 0 0.598" rpy="0 0 0"/>
 </joint>
 <link name="base_link">

Commit message: 更新檔案，移除多餘檔案並新增修改

File: urdf/bipedal_floating.pin.urdf (robot description, URDF)
Before this commit: robot bipedal_floating, 16 links, 15 joints
Joints:
- joint L_Ankle_Pitch: origin xyz=0.0 0.0 -0.2555 rpy=0 0 0 -> xyz=0.0 0.0 -0.2555 rpy=0 -0.37 0
- joint L_Hip_Pitch: origin xyz=0.0 0.032 -0.055 rpy=0 0 0 -> xyz=0.0 0.032 -0.055 rpy=0 -0.37 0
- joint L_Knee_Pitch: origin xyz=0.0 0.019 -0.22 rpy=0 0 0 -> xyz=0.0 0.019 -0.22 rpy=0 0.74 0
- joint R_Ankle_Pitch: origin xyz=0.0 0.0 -0.2555 rpy=0 0 0 -> xyz=0.0 0.0 -0.2555 rpy=0 -0.37 0
- joint R_Hip_Pitch: origin xyz=0.0 -0.032 -0.055 rpy=0 0 0 -> xyz=0.0 -0.032 -0.055 rpy=0 -0.37 0
- joint R_Knee_Pitch: origin xyz=0.0 -0.019 -0.22 rpy=0 0 0 -> xyz=0.0 -0.019 -0.22 rpy=0 0.74 0

File: urdf/bipedal_floating.xacro (robot description, xacro)
@@ -299,5 +299,5 @@
 </joint>
 <joint name="L_Hip_Pitch" type="revolute">
-  <origin xyz="0.0 0.032 -0.055" rpy="0 0 0"/>
+  <origin xyz="0.0 0.032 -0.055" rpy="0 -0.37 0"/>
   <parent link="l_hip_pitch_1"/>
   <child link="l_thigh_1"/>
@@ -307,5 +307,5 @@
 </joint>
 <joint name="L_Knee_Pitch" type="revolute">
-  <origin xyz="0.0 0.019 -0.22" rpy="0 0 0"/>
+  <origin xyz="0.0 0.019 -0.22" rpy="0 0.74 0"/>
   <parent link="l_thigh_1"/>
   <child link="l_shank_1"/>
@@ -315,5 +315,5 @@
 </joint>
 <joint name="L_Ankle_Pitch" type="revolute">
-  <origin xyz="0.0 0.0 -0.2555" rpy="0 0 0"/>
+  <origin xyz="0.0 0.0 -0.2555" rpy="0 -0.37 0"/>
   <parent link="l_shank_1"/>
   <child link="l_ankle_1"/>
@@ -347,5 +347,5 @@
 </joint>
 <joint name="R_Hip_Pitch" type="revolute">
-  <origin xyz="0.0 -0.032 -0.055" rpy="0 0 0"/>
+  <origin xyz="0.0 -0.032 -0.055" rpy="0 -0.37 0"/>
   <parent link="r_hip_pitch_1"/>
   <child link="r_thigh_1"/>
@@ -355,5 +355,5 @@
 </joint>
 <joint name="R_Knee_Pitch" type="revolute">
-  <origin xyz="0.0 -0.019 -0.22" rpy="0 0 0"/>
+  <origin xyz="0.0 -0.019 -0.22" rpy="0 0.74 0"/>
   <parent link="r_thigh_1"/>
   <child link="r_shank_1"/>
@@ -363,5 +363,5 @@
 </joint>
 <joint name="R_Ankle_Pitch" type="revolute">
-  <origin xyz="0.0 0.0 -0.2555" rpy="0 0 0"/>
+  <origin xyz="0.0 0.0 -0.2555" rpy="0 -0.37 0"/>
   <parent link="r_shank_1"/>
   <child link="r_ankle_1"/>

File: urdf/bipedal_l_gravity.xacro (robot description, xacro)
@@ -272,5 +272,5 @@
 </joint>
 <joint name="L_Ankle_Pitch" type="revolute">
-  <origin xyz="0.0 0.0 0.0" rpy="0 0 0"/>
+  <origin xyz="0.0 0.0 0.0" rpy="0 0.37 0"/>
   <parent link="B_UNCA10_ros_v4_1"/>
   <child link="shank_ros_v5_1"/>
@@ -279,5 +279,5 @@
 </joint>
 <joint name="L_Knee_Pitch" type="revolute">
-  <origin xyz="0.0 0.0 0.2555" rpy="0 0 0"/>
+  <origin xyz="0.0 0.0 0.2555" rpy="0 -0.74 0"/>
   <parent link="shank_ros_v5_1"/>
   <child link="thigh_l_ros_v4_1"/>
@@ -286,5 +286,5 @@
 </joint>
 <joint name="L_Hip_Pitch" type="revolute">
-  <origin xyz="0.0 -0.019 0.22" rpy="0 0 0"/>
+  <origin xyz="0.0 -0.019 0.22" rpy="0 0.37 0"/>
   <parent link="thigh_l_ros_v4_1"/>
   <child link="l_hip_pitch_ros_v4_1"/>
@@ -321,5 +321,5 @@
 </joint>
 <joint name="R_Hip_Pitch" type="revolute">
-  <origin xyz="0.0 -0.032 -0.055" rpy="0 0 0"/>
+  <origin xyz="0.0 -0.032 -0.055" rpy="0 -0.37 0"/>
   <parent link="r_hip_pitch_ros_v2_1"/>
   <child link="Thigh_R_v3_1"/>
@@ -328,5 +328,5 @@
 </joint>
 <joint name="R_Knee_Pitch" type="revolute">
-  <origin xyz="0.0 -0.019 -0.22" rpy="0 0 0"/>
+  <origin xyz="0.0 -0.019 -0.22" rpy="0 0.74 0"/>
   <parent link="Thigh_R_v3_1"/>
   <child link="shank_ros_v5__1__1"/>
@@ -335,5 +335,5 @@
 </joint>
 <joint name="R_Ankle_Pitch" type="revolute">
-  <origin xyz="0.0 0.0 -0.2555" rpy="0 0 0"/>
+  <origin xyz="0.0 0.0 -0.2555" rpy="0 -0.37 0"/>
   <parent link="shank_ros_v5__1__1"/>
   <child link="B_UNCA10_ros_v4__1__1"/>

File: urdf/bipedal_r_gravity.xacro (robot description, xacro)
@@ -272,5 +272,5 @@
 </joint>
 <joint name="R_Ankle_Pitch" type="revolute">
-  <origin xyz="0.0 0.0 0.0" rpy="0 0 0"/>
+  <origin xyz="0.0 0.0 0.0" rpy="0 0.37 0"/>
   <parent link="B_UNCA10_ros_v4__1__1"/>
   <child link="shank_ros_v5_1"/>
@@ -279,5 +279,5 @@
 </joint>
 <joint name="R_Knee_Pitch" type="revolute">
-  <origin xyz="0.0 0.0 0.2555" rpy="0 0 0"/>
+  <origin xyz="0.0 0.0 0.2555" rpy="0 -0.74 0"/>
   <parent link="shank_ros_v5_1"/>
   <child link="Thigh_R_v3_1"/>
@@ -286,5 +286,5 @@
 </joint>
 <joint name="R_Hip_Pitch" type="revolute">
-  <origin xyz="0.0 0.019 0.22" rpy="0 0 0"/>
+  <origin xyz="0.0 0.019 0.22" rpy="0 0.37 0"/>
   <parent link="Thigh_R_v3_1"/>
   <child link="r_hip_pitch_ros_v2_1"/>
@@ -321,5 +321,5 @@
 </joint>
 <joint name="L_Hip_Pitch" type="revolute">
-  <origin xyz="0.0 0.032 -0.055" rpy="0 0 0"/>
+  <origin xyz="0.0 0.032 -0.055" rpy="0 -0.37 0"/>
   <parent link="l_hip_pitch_ros_v4_1"/>
   <child link="thigh_l_ros_v4_1"/>
@@ -328,5 +328,5 @@
 </joint>
 <joint name="L_Knee_Pitch" type="revolute">
-  <origin xyz="-0.0 0.019 -0.22" rpy="0 0 0"/>
+  <origin xyz="-0.0 0.019 -0.22" rpy="0 0.74 0"/>
   <parent link="thigh_l_ros_v4_1"/>
   <child link="shank_ros_v5__1__1"/>
@@ -342,5 +342,5 @@
 </joint>
 <joint name="L_Ankle_Roll" type="revolute">
-  <origin xyz="0.0 0.0 0.0" rpy="0 0 0"/>
+  <origin xyz="0.0 0.0 0.0" rpy="0 -0.37 0"/>
   <parent link="B_UNCA10_ros_v4_1"/>
   <child link="footplate_ros_v5__1__1"/>

File: urdf/stance_l.xacro (robot description, xacro)
@@ -154,5 +154,5 @@
 </joint>
 <joint name="L_Ankle_Pitch" type="revolute">
-  <origin xyz="0.0 0.0 0.0" rpy="0 0 0"/>
+  <origin xyz="0.0 0.0 0.0" rpy="0 0.37 0"/>
   <parent link="B_UNCA10_ros_v3_1"/>
   <child link="shank_ros_v4_1"/>
@@ -162,5 +162,5 @@
 </joint>
 <joint name="L_Knee_Pitch" type="revolute">
-  <origin xyz="0.0 0.0 0.2555" rpy="0 0 0"/>
+  <origin xyz="0.0 0.0 0.2555" rpy="0 -0.74 0"/>
   <parent link="shank_ros_v4_1"/>
   <child link="thigh_l_ros_v4_1"/>
@@ -170,5 +170,5 @@
 </joint>
 <joint name="L_Hip_Pitch" type="revolute">
-  <origin xyz="0.0 -0.019 0.22" rpy="0 0 0"/>
+  <origin xyz="0.0 -0.019 0.22" rpy="0 0.37 0"/>
   <parent link="thigh_l_ros_v4_1"/>
   <child link="l_hip_pitch_ros_v4_1"/>

File: urdf/stance_r_gravity.xacro (robot description, xacro)
@@ -152,5 +152,5 @@
 </joint>
 <joint name="R_Ankle_Pitch" type="revolute">
-  <origin xyz="0.0 0.0 0.0" rpy="0 0 0"/>
+  <origin xyz="0.0 0.0 0.0" rpy="0 0.37 0"/>
   <parent link="B_UNCA10_ros_v4_1"/>
   <child link="shank_ros_v5_1"/>
@@ -159,5 +159,5 @@
 </joint>
 <joint name="R_Knee_Pitch" type="revolute">
-  <origin xyz="0.0 0.0 0.2555" rpy="0 0 0"/>
+  <origin xyz="0.0 0.0 0.2555" rpy="0 -0.74 0"/>
   <parent link="shank_ros_v5_1"/>
   <child link="Thigh_R_v3_1"/>
@@ -166,5 +166,5 @@
 </joint>
 <joint name="R_Hip_Pitch" type="revolute">
-  <origin xyz="0.0 0.019 0.22" rpy="0 0 0"/>
+  <origin xyz="0.0 0.019 0.22" rpy="0 0.37 0"/>
   <parent link="Thigh_R_v3_1"/>
   <child link="r_hip_pitch_ros_v2_1"/>

Commit message: <fix>修正角度限制
感謝汪韜學長，雖然我初始角度改了，但角度限制沒有改，所以這之前的版本膝蓋都是無法打直的狀態

File: urdf/bipedal_floating.pin.urdf (robot description, URDF)
Before this commit: robot bipedal_floating, 16 links, 15 joints
Joints:
- joint L_Ankle_Pitch: limit lower=-0.436332 upper=0.436332 effort=100 velocity=100 -> lower=-0.066332 upper=0.806332 effort=100 velocity=100
- joint L_Hip_Pitch: limit lower=-1.570796 upper=1.570796 effort=100 velocity=100 -> lower=-1.200796 upper=1.940796 effort=100 velocity=100
- joint L_Knee_Pitch: limit lower=0.0 upper=1.919862 effort=100 velocity=100 -> lower=-0.74 upper=1.179862 effort=100 velocity=100
- joint R_Ankle_Roll: limit lower=-0.436332 upper=0.436332 effort=100 velocity=100 -> lower=-0.066332 upper=0.806332 effort=100 velocity=100
- joint R_Hip_Pitch: limit lower=-1.570796 upper=1.570796 effort=100 velocity=100 -> lower=-1.200796 upper=1.940796 effort=100 velocity=100
- joint R_Knee_Pitch: limit lower=0.0 upper=1.919862 effort=100 velocity=100 -> lower=-0.74 upper=1.179862 effort=100 velocity=100

File: urdf/bipedal_floating.xacro (robot description, xacro)
@@ -304,5 +304,5 @@
   <axis xyz="0.0 1.0 -0.0"/>
   <dynamics damping="1" friction="0.2"/>
-  <limit upper="1.570796" lower="-1.570796" effort="15" velocity="45"/>
+  <limit upper="1.940796" lower="-1.200796" effort="15" velocity="45"/>
 </joint>
 <joint name="L_Knee_Pitch" type="revolute">
@@ -312,5 +312,5 @@
   <axis xyz="0.0 1.0 0.0"/>
   <dynamics damping="0.25" friction="0.2"/>
-  <limit upper="1.919862" lower="0.0" effort="15" velocity="45"/>
+  <limit upper="1.179862" lower="-0.74" effort="15" velocity="45"/>
 </joint>
 <joint name="L_Ankle_Pitch" type="revolute">
@@ -320,5 +320,5 @@
   <axis xyz="0.0 1.0 0.0"/>
   <dynamics damping="0.05" friction="0.2"/>
-  <limit upper="0.436332" lower="-0.436332" effort="15" velocity="45"/>
+  <limit upper="0.806332" lower="-0.066332" effort="15" velocity="45"/>
 </joint>
 <joint name="L_Ankle_Roll" type="revolute">
@@ -352,5 +352,5 @@
   <axis xyz="0.0 1.0 0.0"/>
   <dynamics damping="1" friction="0.2"/>
-  <limit upper="1.570796" lower="-1.570796" effort="15" velocity="45"/>
+  <limit upper="1.940796" lower="-1.200796" effort="15" velocity="45"/>
 </joint>
 <joint name="R_Knee_Pitch" type="revolute">
@@ -360,5 +360,5 @@
   <axis xyz="0.0 1.0 0.0"/>
   <dynamics damping="0.25" friction="0.2"/>
-  <limit upper="1.919862" lower="0.0" effort="15" velocity="45"/>
+  <limit upper="1.179862" lower="-0.74" effort="15" velocity="45"/>
 </joint>
 <joint name="R_Ankle_Pitch" type="revolute">
@@ -368,5 +368,5 @@
   <axis xyz="0.0 1.0 -0.0"/>
   <dynamics damping="0.05" friction="0.2"/>
-  <limit upper="0.436332" lower="-0.436332" effort="15" velocity="45"/>
+  <limit upper="0.806332" lower="-0.066332" effort="15" velocity="45"/>
 </joint>
 <joint name="R_Ankle_Roll" type="revolute">

Commit message: > urdf改成相對路徑

File: urdf/bipedal_floating.pin.urdf (robot description, URDF)
Before this commit: robot bipedal_floating, 16 links, 15 joints
Links:
- link base_link: geometry collision mesh filename=package://bipedal_floating_description/meshes/base_link.stl scale=0.001 0.001 0.001; visual mesh filename=package://bipedal_floating_description/meshes/base_link.stl scale=0.001 0.001 0.001
- link l_ankle_1: geometry collision mesh filename=package://bipedal_floating_description/meshes/l_ankle_1.stl scale=0.001 0.001 0.001; visual mesh filename=package://bipedal_floating_description/meshes/l_ankle_1.stl scale=0.001 0.001 0.001
- link l_foot_1: geometry collision mesh filename=package://bipedal_floating_description/meshes/l_foot_1.stl scale=0.001 0.001 0.001; visual mesh filename=package://bipedal_floating_description/meshes/l_foot_1.stl scale=0.001 0.001 0.001
- link l_hip_pitch_1: geometry collision mesh filename=package://bipedal_floating_description/meshes/l_hip_pitch_1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 scale=0.001 0.001 0.001; visual mesh filename=package://bipedal_floating_description/meshes/l_hip_pitch_1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 scale=0.001 0.001 0.001
- link l_hip_yaw_1: geometry collision mesh filename=package://bipedal_floating_description/meshes/l_hip_yaw_1.s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 scale=0.001 0.001 0.001; visual mesh filename=package://bipedal_floating_description/meshes/l_hip_yaw_1.s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 scale=0.001 0.001 0.001
- link l_shank_1: geometry collision mesh filename=package://bipedal_floating_description/meshes/l_shank_1.stl scale=0.001 0.001 0.001; visual mesh filename=package://bipedal_floating_description/meshes/l_shank_1.stl scale=0.001 0.001 0.001
- link l_thigh_1: geometry collision mesh filename=package://bipedal_floating_description/meshes/l_thigh_1.stl scale=0.001 0.001 0.001; visual mesh filename=package://bipedal_floating_description/meshes/l_thigh_1.stl scale=0.001 0.001 0.001
- link r_ankle_1: geometry collision mesh filename=package://bipedal_floating_description/meshes/r_ankle_1.stl scale=0.001 0.001 0.001; visual mesh filename=package://bipedal_floating_description/meshes/r_ankle_1.stl scale=0.001 0.001 0.001
- link r_foot_1: geometry collision mesh filename=package://bipedal_floating_description/meshes/r_foot_1.stl scale=0.001 0.001 0.001; visual mesh filename=package://bipedal_floating_description/meshes/r_foot_1.stl scale=0.001 0.001 0.001
- link r_hip_pitch_1: geometry collision mesh filename=package://bipedal_floating_description/meshes/r_hip_pitch_1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 scale=0.001 0.001 0.001; visual mesh filename=package://bipedal_floating_description/meshes/r_hip_pitch_1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 scale=0.001 0.001 0.001
- link r_hip_yaw_1: geometry collision mesh filename=package://bipedal_floating_description/meshes/r_hip_yaw_1.s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 scale=0.001 0.001 0.001; visual mesh filename=package://bipedal_floating_description/meshes/r_hip_yaw_1.s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 scale=0.001 0.001 0.001
- link r_shank_1: geometry collision mesh filename=package://bipedal_floating_description/meshes/r_shank_1.stl scale=0.001 0.001 0.001; visual mesh filename=package://bipedal_floating_description/meshes/r_shank_1.stl scale=0.001 0.001 0.001
- link r_thigh_1: geometry collision mesh filename=package://bipedal_floating_description/meshes/r_thigh_1.stl scale=0.001 0.001 0.001; visual mesh filename=package://bipedal_floating_description/meshes/r_thigh_1.stl scale=0.001 0.001 0.001
